File: mumush.kicad_pcb (KiCad board)
At the start: 2 copper layers, 60 parts, among them J1 Screw_Terminal_01x02, J10 Conn_01x01, J2 header_fan, J3 header_light, J4 Conn_01x01, J5 USB_A, J6 Conn_01x01, J7 Conn_01x01, J8 Conn_01x01, J9 Conn_01x01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

Commit message: PCB progress.
Parts:
- removed the REF** at (52.5, 148.0)
- added REF**: USB_LOGO, myFootprints:USB_LOGO, B.Cu at (124.0, 82.7)
- D1, D2, D3, D4, D5, M1, SW3, SW4, SW5: moved to F.Cu
- J1, J10, J4, J6, J7, J8, J9, U12, U15, U4, U6, U9: moved to B.Cu
- TH1: footprint Connector_JST:JST_XH_B2B-XH-A_1x02_P2.50mm_Vertical -> Connector_PinHeader_2.54mm:PinHeader_1x02_P2.54mm_Horizontal
- U1: footprint Sensor:Aosong_DHT11_5.5x12.0_P2.54mm -> Connector_PinHeader_2.54mm:PinHeader_1x04_P2.54mm_Horizontal
- U5: footprint Connector_PinHeader_2.54mm:PinHeader_1x08_P2.54mm_Vertical -> Connector_PinHeader_2.54mm:PinHeader_1x08_P2.54mm_Horizontal
- moved U8 269.0 mm to (41.4, 143.6), turned to -90 degrees
- moved U1 258.3 mm to (152.8, 148.6), turned to -90 degrees
- moved J5 252.7 mm to (105.2, 145.5)
- moved U5 252.4 mm to (179.9, 148.6), turned to -90 degrees
- moved U10 250.9 mm to (72.5, 141.1), turned to -90 degrees
- moved TH1 249.1 mm to (135.3, 148.3), turned to -90 degrees
- moved R5 246.6 mm to (41.4, 138.6), turned to 180 degrees
- moved J3 245.4 mm to (74.5, 148.2), turned to -90 degrees
- moved J10 241.7 mm to (36.3, 113.2), turned to -90 degrees
- moved J9 240.9 mm to (44.0, 113.2), turned to -90 degrees
- moved U14 236.7 mm to (89.2, 141.2), turned to -90 degrees
- moved R6 236.0 mm to (72.3, 136.0), turned to 180 degrees
- moved R3 234.8 mm to (137.0, 143.6)
- moved C2 233.4 mm to (126.5, 142.4), turned to -90 degrees
- moved SW2 230.5 mm to (89.7, 151.9), turned to 180 degrees
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Connections:
- J2 pad 1: Net-(J2-Pad1) -> +12V
- J2 pad 2: +12V -> Net-(SW1-Pad1)
- SW1 pad 1: Net-(J2-Pad1) -> Net-(SW1-Pad1)
- U4 pad 10: unconnected-(U4-Pad10) -> FAN
- U4 pad 11: unconnected-(U4-Pad11) -> SDA
- U4 pad 14: unconnected-(U4-Pad14) -> SCL
- U4 pad 19: unconnected-(U4-Pad19) -> HEAT
- U4 pad 26: unconnected-(U4-Pad26) -> BTN1
- U4 pad 27: unconnected-(U4-Pad27) -> BTN2
- U4 pad 28: unconnected-(U4-Pad28) -> BTN3
- U4 pad 7: unconnected-(U4-Pad7) -> DHT
- U4 pad 8: unconnected-(U4-Pad8) -> HUMIDIFIER
- U4 pad 9: unconnected-(U4-Pad9) -> LIGHT
Routing:
- net +12V: track 0.00 -> 291.5 mm
- net +3.3V: track 0.00 -> 250.8 mm, vias 0 -> 4
- net SCL: track 0.00 -> 226.4 mm, vias 0 -> 6
- net SDA: track 0.00 -> 206.5 mm, vias 0 -> 6
- net GND: track 0.00 -> 193.3 mm, vias 0 -> 7
- net +5V: track 0.00 -> 184.7 mm, vias 0 -> 2
- net FAN: track 0.00 -> 141.7 mm
- net LIGHT: track 0.00 -> 113.7 mm
- net HUMIDIFIER: track 0.00 -> 104.7 mm
- net HEAT: track 0.00 -> 96.0 mm
- net Net-(SW2-Pad3): track 0.00 -> 95.5 mm, vias 0 -> 2
- net DHT: track 0.00 -> 76.7 mm
- net Net-(SW1-Pad3): track 0.00 -> 76.6 mm
- net Net-(J8-Pad1): track 0.00 -> 67.3 mm
- net Net-(J7-Pad1): track 0.00 -> 54.8 mm
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- added copper zone on B.Cu, net GND
Other:
- board outline added: 194 x 112 mm

Commit message: V1
Parts:
- J5: value USB_A -> humidifier; footprint Connector_USB:USB_A_CONNFLY_DS1095-WNR0 -> Connector_PinHeader_2.54mm:PinHeader_1x02_P2.54mm_Horizontal
- TH1: footprint Connector_PinHeader_2.54mm:PinHeader_1x02_P2.54mm_Horizontal -> Connector_PinHeader_2.54mm:PinHeader_1x02_P2.54mm_Vertical
- U1: footprint Connector_PinHeader_2.54mm:PinHeader_1x04_P2.54mm_Horizontal -> Connector_PinHeader_2.54mm:PinHeader_1x04_P2.54mm_Vertical
- U5: footprint Connector_PinHeader_2.54mm:PinHeader_1x08_P2.54mm_Horizontal -> Connector_PinHeader_2.54mm:PinHeader_1x08_P2.54mm_Vertical
- moved U1 58.2 mm to (115.1, 104.3)
- moved U5 50.4 mm to (132.2, 132.2)
- moved R4 42.6 mm to (124.6, 128.0), turned to 180 degrees
- moved R3 39.2 mm to (115.4, 110.9), turned to 90 degrees
- moved TH1 38.8 mm to (120.1, 112.7), turned to 0 degrees
- moved U3 31.4 mm to (114.3, 116.3), turned to 180 degrees
- moved C2 24.3 mm to (114.1, 121.4), turned to 0 degrees
- moved R7 14.6 mm to (103.8, 136.1)
- moved U14 14.6 mm to (103.8, 141.2)
- moved SW2 14.6 mm to (104.3, 151.9)
- moved J5 14.5 mm to (91.0, 148.2), turned to -90 degrees
Connections:
- J5 pad 1: +5V -> +12V
- J5 pad 2: unconnected-(J5-Pad2) -> Net-(SW2-Pad1)
- SW2 pad 1: Net-(J5-Pad4) -> Net-(SW2-Pad1)
Routing:
- net +5V: track 184.7 -> 49.4 mm, vias 2 -> 0
- net +3.3V: track 250.8 -> 184.5 mm, vias 4 -> 2
- net DHT: track 76.7 -> 16.7 mm
- net SCL: track 226.4 -> 185.0 mm
- net SDA: track 206.5 -> 169.9 mm, vias 6 -> 4
- net Net-(SW2-Pad1): track 0.00 -> 25.5 mm
- net Net-(J5-Pad4): track 24.7 -> 0.00 mm
- net +12V: track 291.5 -> 313.6 mm
- net Net-(SW2-Pad3): track 95.5 -> 117.6 mm
- net GND: track 193.3 -> 174.2 mm
- net FAN: track 141.7 -> 149.5 mm
- net LIGHT: track 113.7 -> 120.4 mm
- net Net-(R4-Pad2): track 5.00 -> 9.98 mm
- net HUMIDIFIER: track 104.7 -> 102.7 mm
Other:
- board text added: "12V"
- board text added: "230~<Fan>12V"
- board text added: "230~<H>12V"
- board text added: "BTN1"
- board text added: "BTN2"
- board text added: "BTN3"
- board text added: "CCS811"
- board text added: "DHT11"
- board text added: "Fan"
- board text added: "GND"
- board text added: "Heat"
- board text added: "Humidifier"
- board text added: "Light"
- board text added: "T°"
